File: Hardware/sparkfun_esp32_environment_sensor_shield.brd (EAGLE design)
At the start: 58.4 x 50.8 mm, 53 parts, among them J1 WEATHER_METER-WIND, J2 WEATHER_METER-RAIN, U1 BME280, U2 CCS811, U3 APDS-9301, U4 TVS Diode

Commit message: Removed restrict layers on antenna for panelization
Parts:
- B1: value ESP32_THING -> ESP32_THING_WO_ANT_KEEPOUT; device SparkFun-Boards:ESP32_THING -> SparkFun-Boards:ESP32_THING_NO_ANT
Changed lines of the file:
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@@
 <layer number="20" name="Dimension" color="15" fill="1" visible="yes" active="yes"/>
 <layer number="21" name="tPlace" color="16" fill="1" visible="yes" active="yes"/>
-<layer number="22" name="bPlace" color="14" fill="1" visible="no" active="yes"/>
+<layer number="22" name="bPlace" color="14" fill="1" visible="yes" active="yes"/>
 <layer number="23" name="tOrigins" color="15" fill="1" visible="yes" active="yes"/>
-<layer number="24" name="bOrigins" color="15" fill="1" visible="no" active="yes"/>
-<layer number="25" name="tNames" color="7" fill="1" visible="yes" active="yes"/>
+<layer number="24" name="bOrigins" color="15" fill="1" visible="yes" active="yes"/>
+<layer number="25" name="tNames" color="7" fill="1" visible="no" active="yes"/>
 <layer number="26" name="bNames" color="7" fill="1" visible="no" active="yes"/>
 <layer number="27" name="tValues" color="7" fill="1" visible="no" active="yes"/>
@@
 <layer number="43" name="vRestrict" color="2" fill="10" visible="no" active="yes"/>
 <layer number="44" name="Drills" color="7" fill="1" visible="no" active="yes"/>
-<layer number="45" name="Holes" color="7" fill="1" visible="no" active="yes"/>
+<layer number="45" name="Holes" color="7" fill="1" visible="yes" active="yes"/>
 <layer number="46" name="Milling" color="3" fill="1" visible="no" active="yes"/>
 <layer number="47" name="Measures" color="7" fill="1" visible="no" active="yes"/>
 <layer number="48" name="Document" color="7" fill="1" visible="no" active="yes"/>
 <layer number="49" name="Reference" color="7" fill="1" visible="no" active="yes"/>
-<layer number="51" name="tDocu" color="6" fill="1" visible="no" active="yes"/>
+<layer number="51" name="tDocu" color="6" fill="1" visible="yes" active="yes"/>
 <layer number="52" name="bDocu" color="7" fill="1" visible="no" active="yes"/>
 <layer number="3" name="Route3" color="4" fill="3" visible="no" active="no"/>
@@
 </autorouter>
 <elements>
-<element name="B1" library="SparkFun-Boards" package="ESP32_THING" value="ESP32_THING" x="16.51" y="0">
-<attribute name="SF_ID" value="DEV-13907" x="16.51" y="0" size="1.778" layer="27" display="off"/>
-</element>
+<element name="B1" library="SparkFun-Boards" package="ESP32_THING_NO_ANT" value="ESP32_THING_WO_ANT_KEEPOUT" x="16.51" y="0"/>
 <element name="FRAME1" library="SparkFun-Aesthetics" package="CREATIVE_COMMONS" value="FRAME-LETTER" x="-13.97" y="-21.59"/>
 <element name="U2" library="esp32-environ-monitor-temp" package="LGA10-2.7X4.0MM" value="CCS811" x="50.8" y="25.4" rot="R90">
@@
 </element>
 <element name="R12" library="esp32-environ-monitor-temp" package="AXIAL-0.1" value="DNP" x="57.15" y="25.4" rot="R270">
-<attribute name="PROD_ID" value="N/A" x="57.15" y="25.4" size="0.8128" layer="27" ratio="15" rot="R270" display="off"/>
 <attribute name="SF_ID" value="SEN-00250" x="57.15" y="25.4" size="1.778" layer="27" rot="R270" display="off"/>
 </element>
